Commit message: showcase for transmissions in mock hw

File: example_8/description/ros2_control/rrbot_transmissions_system_position_only.ros2_control.xacro (robot description, xacro)
@@ -1,8 +1,14 @@
 <?xml version="1.0"?>
 <robot xmlns:xacro="http://www.ros.org/wiki/xacro">
-  <xacro:macro name="rrbot_transmissions_system_position_only" params="name prefix slowdown:=2.0">
+  <xacro:macro name="rrbot_transmissions_system_position_only" params="name prefix slowdown:=^|2.0 use_mock_hardware:=^|false mock_sensor_commands:=^|false">
     <ros2_control name="${name}" type="system">
       <hardware>
-        <plugin>ros2_control_demo_example_8/RRBotTransmissionsSystemPositionOnlyHardware</plugin>
+        <xacro:if value="${use_mock_hardware}">
+          <plugin>mock_components/GenericSystem</plugin>
+          <param name="mock_sensor_commands">${mock_sensor_commands}</param>
+        </xacro:if>
+        <xacro:unless value="${use_mock_hardware}">
+          <plugin>ros2_control_demo_example_8/RRBotTransmissionsSystemPositionOnlyHardware</plugin>
+        </xacro:unless>
         <param name="actuator_slowdown">${slowdown}</param>
       </hardware>
@@ -26,5 +32,5 @@
         <joint name="joint1" role="joint1">
           <mechanical_reduction>2.0</mechanical_reduction>
-          <offset>0.0</offset>
+          <offset>0.2</offset>
         </joint>
       </transmission>
@@ -34,5 +40,5 @@
         <joint name="joint2" role="joint2">
           <mechanical_reduction>4.0</mechanical_reduction>
-          <offset>0.0</offset>
+          <offset>-0.2</offset>
         </joint>
       </transmission>

File: example_8/description/urdf/rrbot_transmissions_system_position_only.urdf.xacro (robot description, xacro)
@@ -9,4 +9,5 @@
   <xacro:arg name="prefix" default="" />
   <xacro:arg name="slowdown" default="100.0" />
+  <xacro:arg name="use_mock_hardware" default="false" />
   <!-- Import RRBot macro -->
   <xacro:include filename="$(find ros2_control_demo_description)/rrbot/urdf/rrbot_description.urdf.xacro" />
@@ -21,5 +22,8 @@
   </xacro:rrbot>
   <xacro:rrbot_transmissions_system_position_only
-    name="RRBotTransmissionsSystemPositionOnly" prefix="$(arg prefix)"
-    slowdown="$(arg slowdown)" />
+    name="RRBotTransmissionsSystemPositionOnly"
+    prefix="$(arg prefix)"
+    slowdown="$(arg slowdown)"
+    use_mock_hardware="$(arg use_mock_hardware)"
+    />
 </robot>
